Commit message: rover design upgrade, rocker-bogie mechanics, solar panel etc

File: robot_description/robot_urdf_description/chassis.xacro (robot description, xacro)
@@ -1,26 +1,29 @@
 <?xml version="1.0"?>
 <robot xmlns:xacro="http://www.ros.org/wiki/xacro">
-    <!-- Chassis dimensions -->
-    <xacro:property name="chassis_length" value="1.5"/>
-    <xacro:property name="chassis_width"  value="1.0"/>
-    <xacro:property name="chassis_height" value="0.3"/>
-    <!-- Chassis mass -->
+    <!-- Main chassis dimensions -->
+    <xacro:property name="chassis_length" value="1.6"/>
+    <xacro:property name="chassis_width" value="1.1"/>
+    <xacro:property name="chassis_height" value="0.30"/>
+    <xacro:property name="chassis_z" value="0.35"/>
     <xacro:property name="chassis_mass" value="20.0"/>
+    <!-- Main body -->
     <link name="base_link">
         <visual>
+            <origin xyz="0 0 ${chassis_z}"/>
             <geometry>
-                <box size="${chassis_length}
-                           ${chassis_width}
-                           ${chassis_height}"/>
+                <box size="${chassis_length} ${chassis_width} ${chassis_height}"/>
             </geometry>
+            <material name="chassis_material">
+                <color rgba="0.18 0.20 0.22 1"/>
+            </material>
         </visual>
         <collision>
+            <origin xyz="0 0 ${chassis_z}"/>
             <geometry>
-                <box size="${chassis_length}
-                           ${chassis_width}
-                           ${chassis_height}"/>
+                <box size="${chassis_length} ${chassis_width} ${chassis_height}"/>
             </geometry>
         </collision>
         <inertial>
+            <origin xyz="0 0 ${chassis_z}"/>
             <mass value="${chassis_mass}"/>
             <inertia
@@ -33,3 +36,37 @@
         </inertial>
     </link>
+    <!-- Raised central equipment deck -->
+    <link name="equipment_deck">
+        <visual>
+            <origin xyz="0 0 0.12"/>
+            <geometry>
+                <box size="1.15 0.80 0.18"/>
+            </geometry>
+            <material name="deck_material">
+                <color rgba="0.25 0.27 0.29 1"/>
+            </material>
+        </visual>
+        <collision>
+            <origin xyz="0 0 0.12"/>
+            <geometry>
+                <box size="1.15 0.80 0.18"/>
+            </geometry>
+        </collision>
+        <inertial>
+            <origin xyz="0 0 0.12"/>
+            <mass value="4.0"/>
+            <inertia
+                ixx="0.2"
+                ixy="0.0"
+                ixz="0.0"
+                iyy="0.2"
+                iyz="0.0"
+                izz="0.2"/>
+        </inertial>
+    </link>
+    <joint name="equipment_deck_joint" type="fixed">
+        <parent link="base_link"/>
+        <child link="equipment_deck"/>
+        <origin xyz="0 0 ${chassis_z + chassis_height/2}"/>
+    </joint>
 </robot>

File: robot_description/robot_urdf_description/robot_body.xacro (robot description, xacro)
@@ -5,3 +5,5 @@
     <xacro:include filename="wheels.xacro"/>
     <xacro:include filename="sensors.xacro"/>
+    <xacro:include filename="solar_panel.xacro"/>
+    <xacro:include filename="details.xacro"/>
 </robot>

File: robot_description/robot_urdf_description/sensors.xacro (robot description, xacro)
@@ -1,21 +1,35 @@
 <?xml version="1.0"?>
 <robot xmlns:xacro="http://www.ros.org/wiki/xacro">
-    <xacro:property name="sensor_mass" value="1.0"/>
+    <!-- ================================================= -->
+    <!-- SENSOR PROPERTIES                                 -->
+    <!-- ================================================= -->
+    <xacro:property name="mast_mass" value="1.0"/>
+    <xacro:property name="head_mass" value="1.5"/>
+    <!-- ================================================= -->
+    <!-- SENSOR MAST                                       -->
+    <!-- ================================================= -->
     <link name="sensor_mast">
         <visual>
-            <origin xyz="0 0 0.25"/>
-            <geometry>
-                <cylinder radius="0.08" length="0.5"/>
-            </geometry>
+            <origin xyz="0 0 0.30"/>
+            <geometry>
+                <cylinder
+                    radius="0.07"
+                    length="0.60"/>
+            </geometry>
+            <material name="mast_material">
+                <color rgba="0.12 0.13 0.14 1"/>
+            </material>
         </visual>
         <collision>
-            <origin xyz="0 0 0.25"/>
-            <geometry>
-                <cylinder radius="0.08" length="0.5"/>
+            <origin xyz="0 0 0.30"/>
+            <geometry>
+                <cylinder
+                    radius="0.07"
+                    length="0.60"/>
             </geometry>
         </collision>
         <inertial>
-            <origin xyz="0 0 0.25"/>
-            <mass value="${sensor_mass}"/>
+            <origin xyz="0 0 0.30"/>
+            <mass value="${mast_mass}"/>
             <inertia
                 ixx="0.02"
@@ -30,5 +44,165 @@
         <parent link="base_link"/>
         <child link="sensor_mast"/>
-        <origin xyz="0 0 0.15"/>
+        <origin
+            xyz="0 0 0.50"
+            rpy="0 0 0"/>
+    </joint>
+    <!-- ================================================= -->
+    <!-- MAIN SENSOR HEAD                                  -->
+    <!-- ================================================= -->
+    <link name="sensor_head">
+        <visual>
+            <geometry>
+                <box size="0.45 0.30 0.20"/>
+            </geometry>
+            <material name="sensor_head_material">
+                <color rgba="0.16 0.17 0.18 1"/>
+            </material>
+        </visual>
+        <collision>
+            <geometry>
+                <box size="0.45 0.30 0.20"/>
+            </geometry>
+        </collision>
+        <inertial>
+            <mass value="${head_mass}"/>
+            <inertia
+                ixx="0.03"
+                ixy="0.0"
+                ixz="0.0"
+                iyy="0.03"
+                iyz="0.0"
+                izz="0.03"/>
+        </inertial>
+    </link>
+    <joint name="sensor_head_joint" type="fixed">
+        <parent link="sensor_mast"/>
+        <child link="sensor_head"/>
+        <origin
+            xyz="0 0 0.65"
+            rpy="0 0 0"/>
+    </joint>
+    <!-- ================================================= -->
+    <!-- LEFT CAMERA HOUSING                               -->
+    <!-- ================================================= -->
+    <link name="left_camera">
+        <visual>
+            <origin xyz="0 0 0"/>
+            <geometry>
+                <box size="0.12 0.10 0.10"/>
+            </geometry>
+            <material name="camera_housing_material">
+                <color rgba="0.08 0.09 0.10 1"/>
+            </material>
+        </visual>
+    </link>
+    <joint name="left_camera_joint" type="fixed">
+        <parent link="sensor_head"/>
+        <child link="left_camera"/>
+        <origin
+            xyz="0.235 0.085 0.025"
+            rpy="0 0 0"/>
+    </joint>
+    <!-- Left camera lens -->
+    <link name="left_camera_lens">
+        <visual>
+            <origin xyz="0 0 0"/>
+            <geometry>
+                <cylinder
+                    radius="0.035"
+                    length="0.025"/>
+            </geometry>
+            <material name="lens_material">
+                <color rgba="0.02 0.05 0.08 1"/>
+            </material>
+        </visual>
+    </link>
+    <joint name="left_camera_lens_joint" type="fixed">
+        <parent link="left_camera"/>
+        <child link="left_camera_lens"/>
+        <origin
+            xyz="0.065 0 0"
+            rpy="0 1.5708 0"/>
+    </joint>
+    <!-- ================================================= -->
+    <!-- RIGHT CAMERA HOUSING                              -->
+    <!-- ================================================= -->
+    <link name="right_camera">
+        <visual>
+            <geometry>
+                <box size="0.12 0.10 0.10"/>
+            </geometry>
+            <material name="camera_housing_material"/>
+        </visual>
+    </link>
+    <joint name="right_camera_joint" type="fixed">
+        <parent link="sensor_head"/>
+        <child link="right_camera"/>
+        <origin
+            xyz="0.235 -0.085 0.025"
+            rpy="0 0 0"/>
+    </joint>
+    <!-- Right camera lens -->
+    <link name="right_camera_lens">
+        <visual>
+            <geometry>
+                <cylinder
+                    radius="0.035"
+                    length="0.025"/>
+            </geometry>
+            <material name="lens_material"/>
+        </visual>
+    </link>
+    <joint name="right_camera_lens_joint" type="fixed">
+        <parent link="right_camera"/>
+        <child link="right_camera_lens"/>
+        <origin
+            xyz="0.065 0 0"
+            rpy="0 1.5708 0"/>
+    </joint>
+    <!-- ================================================= -->
+    <!-- CENTRAL RANGE SENSOR                               -->
+    <!-- ================================================= -->
+    <link name="range_sensor">
+        <visual>
+            <origin xyz="0 0 0"/>
+            <geometry>
+                <cylinder
+                    radius="0.055"
+                    length="0.04"/>
+            </geometry>
+            <material name="range_sensor_material">
+                <color rgba="0.03 0.04 0.05 1"/>
+            </material>
+        </visual>
+    </link>
+    <joint name="range_sensor_joint" type="fixed">
+        <parent link="sensor_head"/>
+        <child link="range_sensor"/>
+        <origin
+            xyz="0.235 0 -0.055"
+            rpy="0 1.5708 0"/>
+    </joint>
+    <!-- ================================================= -->
+    <!-- TOP SENSOR                                         -->
+    <!-- ================================================= -->
+    <link name="top_sensor">
+        <visual>
+            <geometry>
+                <cylinder
+                    radius="0.06"
+                    length="0.08"/>
+            </geometry>
+            <material name="top_sensor_material">
+                <color rgba="0.25 0.26 0.27 1"/>
+            </material>
+        </visual>
+    </link>
+    <joint name="top_sensor_joint" type="fixed">
+        <parent link="sensor_head"/>
+        <child link="top_sensor"/>
+        <origin
+            xyz="-0.05 0 0.14"
+            rpy="0 0 0"/>
     </joint>
 </robot>

File: robot_description/robot_urdf_description/wheels.xacro (robot description, xacro)
@@ -1,10 +1,16 @@
 <?xml version="1.0"?>
 <robot xmlns:xacro="http://www.ros.org/wiki/xacro">
+    <!-- ================================================= -->
+    <!-- WHEEL PROPERTIES                                  -->
+    <!-- ================================================= -->
     <xacro:property name="wheel_radius" value="0.25"/>
     <xacro:property name="wheel_width" value="0.15"/>
     <xacro:property name="wheel_mass" value="2.0"/>
-    <!-- Wheel geometry -->
+    <!-- ================================================= -->
+    <!-- WHEEL MACRO                                       -->
+    <!-- ================================================= -->
     <xacro:macro name="wheel" params="name x y">
         <link name="${name}">
+            <!-- Tire -->
             <visual>
                 <origin rpy="1.5708 0 0"/>
@@ -14,5 +20,9 @@
                         length="${wheel_width}"/>
                 </geometry>
+                <material name="wheel_material">
+                    <color rgba="0.08 0.08 0.08 1"/>
+                </material>
             </visual>
+            <!-- Tire collision -->
             <collision>
                 <origin rpy="1.5708 0 0"/>
@@ -23,4 +33,5 @@
                 </geometry>
             </collision>
+            <!-- Wheel mass -->
             <inertial>
                 <mass value="${wheel_mass}"/>
@@ -34,18 +45,237 @@
             </inertial>
         </link>
-        <joint name="${name}_joint" type="continuous">
+        <!-- Wheel axle -->
+        <joint
+            name="${name}_joint"
+            type="continuous">
             <parent link="base_link"/>
             <child link="${name}"/>
-            <origin xyz="${x} ${y} 0.0" rpy="0 0 0"/>
+            <origin
+                xyz="${x} ${y} 0"
+                rpy="0 0 0"/>
             <axis xyz="0 1 0"/>
         </joint>
     </xacro:macro>
-    <!-- Left side -->
-    <xacro:wheel name="front_left_wheel"  x="0.55"  y="0.55"/>
-    <xacro:wheel name="middle_left_wheel" x="0.0"   y="0.55"/>
-    <xacro:wheel name="rear_left_wheel"   x="-0.55" y="0.55"/>
-    <!-- Right side -->
-    <xacro:wheel name="front_right_wheel"  x="0.55"  y="-0.55"/>
-    <xacro:wheel name="middle_right_wheel" x="0.0"   y="-0.55"/>
-    <xacro:wheel name="rear_right_wheel"   x="-0.55" y="-0.55"/>
+    <!-- ================================================= -->
+    <!-- SIX WHEELS                                        -->
+    <!-- ================================================= -->
+    <!-- LEFT -->
+    <xacro:wheel
+        name="front_left_wheel"
+        x="0.55"
+        y="0.62"/>
+    <xacro:wheel
+        name="middle_left_wheel"
+        x="0.0"
+        y="0.62"/>
+    <xacro:wheel
+        name="rear_left_wheel"
+        x="-0.55"
+        y="0.62"/>
+    <!-- RIGHT -->
+    <xacro:wheel
+        name="front_right_wheel"
+        x="0.55"
+        y="-0.62"/>
+    <xacro:wheel
+        name="middle_right_wheel"
+        x="0.0"
+        y="-0.62"/>
+    <xacro:wheel
+        name="rear_right_wheel"
+        x="-0.55"
+        y="-0.62"/>
+    <!-- ================================================= -->
+    <!-- ROCKER-BOGIE VISUAL STRUCTURE                    -->
+    <!-- ================================================= -->
+    <!-- ================================================= -->
+    <!-- LEFT ROCKER                                      -->
+    <!-- ================================================= -->
+    <link name="left_rocker">
+        <visual>
+            <!-- Long arm running toward front wheel -->
+            <origin
+                xyz="0.25 0 0.02"
+                rpy="0 -0.08 0"/>
+            <geometry>
+                <box size="0.65 0.14 0.16"/>
+            </geometry>
+            <material name="suspension_material">
+                <color rgba="0.28 0.29 0.30 1"/>
+            </material>
+        </visual>
+    </link>
+    <joint name="left_rocker_joint" type="fixed">
+        <parent link="base_link"/>
+        <child link="left_rocker"/>
+        <origin
+            xyz="0 0.62 0.18"
+            rpy="0 0 0"/>
+    </joint>
+    <!-- ================================================= -->
+    <!-- RIGHT ROCKER                                     -->
+    <!-- ================================================= -->
+    <link name="right_rocker">
+        <visual>
+            <origin
+                xyz="0.25 0 0.02"
+                rpy="0 -0.08 0"/>
+            <geometry>
+                <box size="0.65 0.14 0.16"/>
+            </geometry>
+            <material name="suspension_material"/>
+        </visual>
+    </link>
+    <joint name="right_rocker_joint" type="fixed">
+        <parent link="base_link"/>
+        <child link="right_rocker"/>
+        <origin
+            xyz="0 -0.62 0.18"
+            rpy="0 0 0"/>
+    </joint>
+    <!-- ================================================= -->
+    <!-- LEFT BOGIE                                       -->
+    <!-- ================================================= -->
+    <link name="left_bogie">
+        <visual>
+            <!-- Arm running from middle toward rear -->
+            <origin
+                xyz="-0.27 0 -0.05"
+                rpy="0 0.15 0"/>
+            <geometry>
+                <box size="0.70 0.14 0.16"/>
+            </geometry>
+            <material name="suspension_material"/>
+        </visual>
+    </link>
+    <joint name="left_bogie_joint" type="fixed">
+        <parent link="base_link"/>
+        <child link="left_bogie"/>
+        <origin
+            xyz="0 0.62 0.12"
+            rpy="0 0 0"/>
+    </joint>
+    <!-- ================================================= -->
+    <!-- RIGHT BOGIE                                      -->
+    <!-- ================================================= -->
+    <link name="right_bogie">
+        <visual>
+            <origin
+                xyz="-0.27 0 -0.05"
+                rpy="0 0.15 0"/>
+            <geometry>
+                <box size="0.70 0.14 0.16"/>
+            </geometry>
+            <material name="suspension_material"/>
+        </visual>
+    </link>
+    <joint name="right_bogie_joint" type="fixed">
+        <parent link="base_link"/>
+        <child link="right_bogie"/>
+        <origin
+            xyz="0 -0.62 0.12"
+            rpy="0 0 0"/>
+    </joint>
+    <!-- ================================================= -->
+    <!-- FRONT SUSPENSION MOUNTS                          -->
+    <!-- ================================================= -->
+    <link name="front_left_mount">
+        <visual>
+            <origin xyz="0 0 0.02"/>
+            <geometry>
+                <box size="0.14 0.18 0.30"/>
+            </geometry>
+            <material name="suspension_material"/>
+        </visual>
+    </link>
+    <joint name="front_left_mount_joint" type="fixed">
+        <parent link="base_link"/>
+        <child link="front_left_mount"/>
+        <origin
+            xyz="0.55 0.62 0.02"
+            rpy="0 0 0"/>
+    </joint>
+    <link name="front_right_mount">
+        <visual>
+            <origin xyz="0 0 0.02"/>
+            <geometry>
+                <box size="0.14 0.18 0.30"/>
+            </geometry>
+            <material name="suspension_material"/>
+        </visual>
+    </link>
+    <joint name="front_right_mount_joint" type="fixed">
+        <parent link="base_link"/>
+        <child link="front_right_mount"/>
+        <origin
+            xyz="0.55 -0.62 0.02"
+            rpy="0 0 0"/>
+    </joint>
+    <!-- ================================================= -->
+    <!-- REAR SUSPENSION MOUNTS                           -->
+    <!-- ================================================= -->
+    <link name="rear_left_mount">
+        <visual>
+            <origin xyz="0 0 0.02"/>
+            <geometry>
+                <box size="0.14 0.18 0.30"/>
+            </geometry>
+            <material name="suspension_material"/>
+        </visual>
+    </link>
+    <joint name="rear_left_mount_joint" type="fixed">
+        <parent link="base_link"/>
+        <child link="rear_left_mount"/>
+        <origin
+            xyz="-0.55 0.62 0.02"
+            rpy="0 0 0"/>
+    </joint>
+    <link name="rear_right_mount">
+        <visual>
+            <origin xyz="0 0 0.02"/>
+            <geometry>
+                <box size="0.14 0.18 0.30"/>
+            </geometry>
+            <material name="suspension_material"/>
+        </visual>
+    </link>
+    <joint name="rear_right_mount_joint" type="fixed">
+        <parent link="base_link"/>
+        <child link="rear_right_mount"/>
+        <origin
+            xyz="-0.55 -0.62 0.02"
+            rpy="0 0 0"/>
+    </joint>
+    <!-- ================================================= -->
+    <!-- WHEEL HUBS                                       -->
+    <!-- ================================================= -->
+    <xacro:macro name="wheel_hub" params="name x y">
+        <link name="${name}_hub">
+            <visual>
+                <origin rpy="1.5708 0 0"/>
+                <geometry>
+                    <cylinder
+                        radius="0.11"
+                        length="0.18"/>
+                </geometry>
+                <material name="hub_material">
+                    <color rgba="0.35 0.36 0.37 1"/>
+                </material>
+            </visual>
+        </link>
+        <joint name="${name}_hub_joint" type="fixed">
+            <parent link="base_link"/>
+            <child link="${name}_hub"/>
+            <origin
+                xyz="${x} ${y} 0"
+                rpy="0 0 0"/>
+        </joint>
+    </xacro:macro>
+    <!-- Hubs -->
+    <xacro:wheel_hub name="front_left_wheel" x="0.55" y="0.62"/>
+    <xacro:wheel_hub name="middle_left_wheel" x="0.0" y="0.62"/>
+    <xacro:wheel_hub name="rear_left_wheel" x="-0.55" y="0.62"/>
+    <xacro:wheel_hub name="front_right_wheel" x="0.55" y="-0.62"/>
+    <xacro:wheel_hub name="middle_right_wheel" x="0.0" y="-0.62"/>
+    <xacro:wheel_hub name="rear_right_wheel" x="-0.55" y="-0.62"/>
 </robot>
