Commit message: gazebo actuation, yaml file for controllers added

File: robot_description/robot_urdf_description/robot_body.xacro (robot description, xacro)
@@ -7,3 +7,46 @@
     <xacro:include filename="solar_panel.xacro"/>
     <xacro:include filename="details.xacro"/>
+    <!-- Simulated wheel hardware interface -->
+    <ros2_control name="RoverDriveSystem" type="system">
+        <hardware>
+            <plugin>gz_ros2_control/GazeboSimSystem</plugin>
+        </hardware>
+        <joint name="front_left_wheel_joint">
+            <command_interface name="velocity"/>
+            <state_interface name="position"/>
+            <state_interface name="velocity"/>
+        </joint>
+        <joint name="middle_left_wheel_joint">
+            <command_interface name="velocity"/>
+            <state_interface name="position"/>
+            <state_interface name="velocity"/>
+        </joint>
+        <joint name="rear_left_wheel_joint">
+            <command_interface name="velocity"/>
+            <state_interface name="position"/>
+            <state_interface name="velocity"/>
+        </joint>
+        <joint name="front_right_wheel_joint">
+            <command_interface name="velocity"/>
+            <state_interface name="position"/>
+            <state_interface name="velocity"/>
+        </joint>
+        <joint name="middle_right_wheel_joint">
+            <command_interface name="velocity"/>
+            <state_interface name="position"/>
+            <state_interface name="velocity"/>
+        </joint>
+        <joint name="rear_right_wheel_joint">
+            <command_interface name="velocity"/>
+            <state_interface name="position"/>
+            <state_interface name="velocity"/>
+        </joint>
+    </ros2_control>
+    <!-- Gazebo ROS 2 control plugin -->
+    <gazebo>
+        <plugin filename="gz_ros2_control-system"
+                name="gz_ros2_control::GazeboSimROS2ControlPlugin">
+            <parameters>$(find rover_gazebo)/config/controllers.yaml</parameters>
+        </plugin>
+    </gazebo>
 </robot>

File: robot_description/robot_urdf_description/wheels.xacro (robot description, xacro)
@@ -37,10 +37,10 @@
                 <mass value="${wheel_mass}"/>
                 <inertia
-                    ixx="0.1"
+                    ixx="0.035"
                     ixy="0.0"
                     ixz="0.0"
-                    iyy="0.1"
+                    iyy="0.0625"
                     iyz="0.0"
-                    izz="0.1"/>
+                    izz="0.035"/>
             </inertial>
         </link>
