Commit message: configured lidar sensor to robot description

File: robot_description/robot_urdf_description/sensors.xacro (robot description, xacro)
@@ -206,3 +206,66 @@
             rpy="0 0 0"/>
     </joint>
+    <!-- ================================================= -->
+    <!-- 3D LIDAR SENSOR                                   -->
+    <!-- ================================================= -->
+    <link name="lidar_link">
+        <visual>
+            <geometry>
+                <cylinder radius="0.08" length="0.06"/>
+            </geometry>
+            <material name="lidar_material">
+                <color rgba="0.08 0.08 0.09 1"/>
+            </material>
+        </visual>
+        <collision>
+            <geometry>
+                <cylinder radius="0.08" length="0.06"/>
+            </geometry>
+        </collision>
+        <inertial>
+            <mass value="0.3"/>
+            <inertia
+                ixx="0.0005"
+                ixy="0.0"
+                ixz="0.0"
+                iyy="0.0005"
+                iyz="0.0"
+                izz="0.0008"/>
+        </inertial>
+    </link>
+    <joint name="lidar_joint" type="fixed">
+        <parent link="sensor_head"/>
+        <child link="lidar_link"/>
+        <origin xyz="0 0 0.17" rpy="0 0 0"/>
+    </joint>
+    <gazebo reference="lidar_link">
+        <sensor name="lidar_link" type="gpu_lidar">
+            <pose>0 0 0 0 0 0</pose>
+            <topic> /lidar/scan </topic>
+            <update_rate>10</update_rate>
+            <lidar>
+                <scan>
+                    <horizontal>
+                        <samples>360</samples>
+                        <resolution>1</resolution>
+                        <min_angle>-3.14159</min_angle>
+                        <max_angle>3.14159</max_angle>
+                    </horizontal>
+                    <vertical>
+                        <samples>16</samples>
+                        <resolution>1</resolution>
+                        <min_angle>-0.2618</min_angle>
+                        <max_angle>0.2618</max_angle>
+                    </vertical>
+                </scan>
+                <range>
+                    <min>0.1</min>
+                    <max>20.0</max>
+                    <resolution>0.01</resolution>
+                </range>
+            </lidar>
+            <always_on>true</always_on>
+            <visualize>true</visualize>
+        </sensor>
+    </gazebo>
 </robot>
